File: Laser_Diode_Driver.kicad_pcb (KiCad board)
At the start: 2 copper layers, 21.5 x 12.5 mm, 7 parts, among them J1 Conn_01x02, Q1 SS8050, Q2 S8050, SW1 SW_Push

Commit message: fix: small modification on the silkscreen for information.
Other:
- board text added: "- +"
